Commit message: Gazeboシミュレータ機能を実装

File: amir_description/urdf/amir_for_rover.xacro (robot description, xacro)
@@ -6,7 +6,12 @@
 <link name="link0_1">
   <inertial>
-    <origin xyz="-0.00035733615838378973 -0.01841918266108223 -0.16514949503635634" rpy="0 0 0"/>
-    <mass value="5.57955152018178"/>
-    <inertia ixx="0.026615" iyy="0.023143" izz="0.022213" ixy="-1e-06" iyz="-0.000292" ixz="1e-06"/>
+    <origin xyz="0.0 -0.018171 -0.164351" rpy="0 0 0"/>
+    <mass value="2.37148"/>
+    <inertia ixx="0.01020"
+             iyy="0.008745"
+             izz="0.008637"
+             ixy="-0.000000291275"
+             iyz="-0.0001135"
+             ixz="0.000000428733"/>
   </inertial>
   <visual>
@@ -26,10 +31,15 @@
 <link name="link1_1">
   <inertial>
-    <origin xyz="-0.00018985799062385848 -0.020942565042805037 0.039786642292211995" rpy="0 0 0"/>
-    <mass value="3.561104838398658"/>
-    <inertia ixx="0.010766" iyy="0.010657" izz="0.012144" ixy="-0.000403" iyz="-0.000117" ixz="-0.000406"/>
-  </inertial>
-  <visual>
-    <origin xyz="0.000367 0.001523 0.097" rpy="0 0 0"/>
+    <origin xyz="0.00 -0.015481739081542548 0.052015680869348734" rpy="0 0 0"/>
+    <mass value="1.530171"/>
+    <inertia ixx="0.003518"
+             iyy="0.003654"
+             izz="0.004561"
+             ixy="0.0002342"
+             iyz="0.00002134302"
+             ixz="-0.000060488629"/>
+  </inertial>
+  <visual>
+    <origin xyz="0.00 0.001523 0.097" rpy="0 0 0"/>
     <geometry>
       <mesh filename="package://amir_description/meshes/link1_1.stl" scale="0.001 0.001 0.001"/>
@@ -38,5 +48,5 @@
   </visual>
   <collision>
-    <origin xyz="0.000367 0.001523 0.097" rpy="0 0 0"/>
+    <origin xyz="0.00 0.001523 0.097" rpy="0 0 0"/>
     <geometry>
       <mesh filename="package://amir_description/meshes/link1_1.stl" scale="0.001 0.001 0.001"/>
@@ -46,10 +56,15 @@
 <link name="link2_1">
   <inertial>
-    <origin xyz="0.034529749920508966 0.10697083960868432 0.009616079185851476" rpy="0 0 0"/>
-    <mass value="3.718072990915677"/>
-    <inertia ixx="0.04067" iyy="0.008258" izz="0.046013" ixy="0.000387" iyz="-0.001192" ixz="0.000332"/>
-  </inertial>
-  <visual>
-    <origin xyz="0.034367 0.001523 -0.0" rpy="0 0 0"/>
+    <origin xyz="0.00 0.13301271963728503 0.014415028610505691" rpy="0 0 0"/>
+    <mass value="1.863224"/>
+    <inertia ixx="0.01781"
+             iyy="0.003563"
+             izz="0.02037"
+             ixy="0.002226"
+             iyz="-0.0008328"
+             ixz="0.0002878"/>
+  </inertial>
+  <visual>
+    <origin xyz="0.0 0.001523 -0.0" rpy="0 0 0"/>
     <geometry>
       <mesh filename="package://amir_description/meshes/link2_1.stl" scale="0.001 0.001 0.001"/>
@@ -58,5 +73,5 @@
   </visual>
   <collision>
-    <origin xyz="0.034367 0.001523 -0.0" rpy="0 0 0"/>
+    <origin xyz="0.0 0.001523 -0.0" rpy="0 0 0"/>
     <geometry>
       <mesh filename="package://amir_description/meshes/link2_1.stl" scale="0.001 0.001 0.001"/>
@@ -66,10 +81,15 @@
 <link name="link3_1">
   <inertial>
-    <origin xyz="0.04147569573190948 0.10393679437717612 0.009489090607211592" rpy="0 0 0"/>
-    <mass value="2.387172799459861"/>
-    <inertia ixx="0.034538" iyy="0.002646" izz="0.034829" ixy="0.000602" iyz="-0.001389" ixz="0.000136"/>
-  </inertial>
-  <visual>
-    <origin xyz="0.034367 -0.308477 0.000172" rpy="0 0 0"/>
+    <origin xyz="-0.0 0.11541444998364736 0.013649097933998836" rpy="0 0 0"/>
+    <mass value="0.904315"/>
+    <inertia ixx="0.01374"
+             iyy="0.0009585"
+             izz="0.01392"
+             ixy="0.0004506"
+             iyz="-0.0007046"
+             ixz="0.000064200508"/>
+  </inertial>
+  <visual>
+    <origin xyz="-0.0 -0.308477 0.0" rpy="0 0 0"/>
     <geometry>
       <mesh filename="package://amir_description/meshes/link3_1.stl" scale="0.001 0.001 0.001"/>
@@ -78,5 +98,5 @@
   </visual>
   <collision>
-    <origin xyz="0.034367 -0.308477 0.000172" rpy="0 0 0"/>
+    <origin xyz="-0.0 -0.308477 0.0" rpy="0 0 0"/>
     <geometry>
       <mesh filename="package://amir_description/meshes/link3_1.stl" scale="0.001 0.001 0.001"/>
@@ -86,10 +106,15 @@
 <link name="link4_1">
   <inertial>
-    <origin xyz="0.03766898869025648 0.0016682567902981393 -1.7795557616154505e-05" rpy="0 0 0"/>
-    <mass value="0.7997873584496068"/>
-    <inertia ixx="0.000517" iyy="0.000449" izz="0.000488" ixy="1.2e-05" iyz="0.0" ixz="0.0"/>
-  </inertial>
-  <visual>
-    <origin xyz="0.030367 -0.618476 -0.000403" rpy="0 0 0"/>
+    <origin xyz="0.0 0.002871377179418988 -2.4706069597529916e-10" rpy="0 0 0"/>
+    <mass value="0.261183"/>
+    <inertia ixx="0.000153"
+             iyy="0.000144"
+             izz="0.0001626"
+             ixy="0.000007504862"
+             iyz="-0.000000008483"
+             ixz="-0.000000007056"/>
+  </inertial>
+  <visual>
+    <origin xyz="0.0 -0.618477 -0.0" rpy="0 0 0"/>
     <geometry>
       <mesh filename="package://amir_description/meshes/link4_1.stl" scale="0.001 0.001 0.001"/>
@@ -98,5 +123,5 @@
   </visual>
   <collision>
-    <origin xyz="0.030367 -0.618476 -0.000403" rpy="0 0 0"/>
+    <origin xyz="0.0 -0.618477 -0.0" rpy="0 0 0"/>
     <geometry>
       <mesh filename="package://amir_description/meshes/link4_1.stl" scale="0.001 0.001 0.001"/>
@@ -104,13 +129,33 @@
   </collision>
 </link>
-<link name="link5_1" />
+<!-- add tool center point link for easier visualization -->
+<link name="tcp_link">
+  <visual>
+    <geometry>
+      <box size="0.01 0.01 0.01"/>
+    </geometry>
+    <material name="red">
+      <color rgba="1.0 0.0 0.0 0.6"/>
+    </material>
+  </visual>
+</link>
+<joint name="tcp_fixed" type="fixed">
+  <origin xyz="0.0 0.0795 0.0" rpy="0 0 0"/>
+  <parent link="gripper_base_1"/>
+  <child link="tcp_link"/>
+</joint>
 <link name="gripper_base_1">
   <inertial>
-    <origin xyz="0.00880330299144775 0.01811292766821604 -0.00366390127533253" rpy="0 0 0"/>
-    <mass value="0.30983997234277605"/>
-    <inertia ixx="0.000178" iyy="0.000255" izz="0.000135" ixy="-7e-06" iyz="4e-06" ixz="4e-06"/>
-  </inertial>
-  <visual>
-    <origin xyz="0.000367 -0.656976 -0.000403" rpy="0 0 0"/>
+    <origin xyz="0.0 0.01128514374633649 -0.004836003736858561" rpy="0 0 0"/>
+    <mass value="0.130337"/>
+    <inertia ixx="0.00008551164"
+             iyy="0.0001216"
+             izz="0.000059771966"
+             ixy="-0.000003161031"
+             iyz="0.000001110492"
+             ixz="-0.000003519581"/>
+  </inertial>
+  <visual>
+    <origin xyz="0.0 -0.658977 -0.0" rpy="0 0 0"/>
     <geometry>
       <mesh filename="package://amir_description/meshes/gripper_base_1.stl" scale="0.001 0.001 0.001"/>
@@ -119,5 +164,5 @@
   </visual>
   <collision>
-    <origin xyz="0.000367 -0.656976 -0.000403" rpy="0 0 0"/>
+    <origin xyz="0.0 -0.658977 -0.0" rpy="0 0 0"/>
     <geometry>
       <mesh filename="package://amir_description/meshes/gripper_base_1.stl" scale="0.001 0.001 0.001"/>
@@ -125,12 +170,188 @@
   </collision>
 </link>
+<link name="inner_link_left_1">
+  <inertial>
+    <origin xyz="0.004775263006022466 0.014691054356398392 0.0" rpy="0 0 0"/>
+    <mass value="0.010214"/>
+    <inertia ixx="0.000007990586"
+             iyy="0.000005973968"
+             izz="0.000002702176"
+             ixy="-0.000000446816"
+             iyz="0.0000"
+             ixz="-0.00000"/>
+  </inertial>
+  <visual>
+    <origin xyz="0.018 -0.679499 -0.0" rpy="0 0 0"/>
+    <geometry>
+      <mesh filename="package://amir_description/meshes/inner_link_left_1.stl" scale="0.001 0.001 0.001"/>
+    </geometry>
+    <material name="silver-amir"/>
+  </visual>
+  <collision>
+    <origin xyz="0.018 -0.679499 -0.0" rpy="0 0 0"/>
+    <geometry>
+      <mesh filename="package://amir_description/meshes/inner_link_left_1.stl" scale="0.001 0.001 0.001"/>
+    </geometry>
+  </collision>
+</link>
+<link name="outer_link_right_1">
+  <inertial>
+    <origin xyz="0.0029741808490290345 0.020000417105897617 0.0" rpy="0 0 0"/>
+    <mass value="0.015216"/>
+    <inertia ixx="0.000009064719"
+             iyy="0.000006207691"
+             izz="0.000003674706"
+             ixy="0.000000861905"
+             iyz="-0.0"
+             ixz="0.0"/>
+  </inertial>
+  <visual>
+    <origin xyz="-0.038 -0.679499 -0.0" rpy="0 0 0"/>
+    <geometry>
+      <mesh filename="package://amir_description/meshes/outer_link_right_1.stl" scale="0.001 0.001 0.001"/>
+    </geometry>
+    <material name="silver-amir"/>
+  </visual>
+  <collision>
+    <origin xyz="-0.038 -0.679499 -0.0" rpy="0 0 0"/>
+    <geometry>
+      <mesh filename="package://amir_description/meshes/outer_link_right_1.stl" scale="0.001 0.001 0.001"/>
+    </geometry>
+  </collision>
+</link>
+<link name="outer_link_left_1">
+  <inertial>
+    <origin xyz="-0.002974180849028861 0.020000417105899837 0.0" rpy="0 0 0"/>
+    <mass value="0.015216"/>
+    <inertia ixx="0.000009073869"
+             iyy="0.000006198542"
+             izz="0.000003674706"
+             ixy="-0.000000846555"
+             iyz="0.00000"
+             ixz="0.00000"/>
+  </inertial>
+  <visual>
+    <origin xyz="0.038 -0.679499 -0.0" rpy="0 0 0"/>
+    <geometry>
+      <mesh filename="package://amir_description/meshes/outer_link_left_1.stl" scale="0.001 0.001 0.001"/>
+    </geometry>
+    <material name="silver-amir"/>
+  </visual>
+  <collision>
+    <origin xyz="0.038 -0.679499 -0.0" rpy="0 0 0"/>
+    <geometry>
+      <mesh filename="package://amir_description/meshes/outer_link_left_1.stl" scale="0.001 0.001 0.001"/>
+    </geometry>
+  </collision>
+</link>
+<!-- NOTE: urdf doesnt support kinematic closed loop,
+so we need to left one on the joints open -->
+<!-- use this when using inner link -->
+<link name="finger_right_1">
+  <inertial>
+    <origin xyz="0.002489444086893569 0.012411313372935995 0.0" rpy="0 0 0"/>
+    <mass value="0.022898"/>
+    <inertia ixx="0.000017128826"
+             iyy="0.000011930401"
+             izz="0.000008715513"
+             ixy="0.000001953953"
+             iyz="0.00"
+             ixz="-0.00"/>
+  </inertial>
+  <visual>
+    <origin xyz="-0.018 -0.719499 -0.0" rpy="0 0 0"/>
+    <geometry>
+      <mesh filename="package://amir_description/meshes/finger_right_1.stl" scale="0.001 0.001 0.001"/>
+    </geometry>
+    <material name="silver-amir"/>
+  </visual>
+  <collision>
+    <origin xyz="-0.018 -0.719499 -0.0" rpy="0 0 0"/>
+    <geometry>
+      <mesh filename="package://amir_description/meshes/finger_right_1.stl" scale="0.001 0.001 0.001"/>
+    </geometry>
+  </collision>
+</link>
+<link name="finger_left_1">
+  <inertial>
+    <origin xyz="-0.0024894440868974757 0.012411313372938326 0.0" rpy="0 0 0"/>
+    <mass value="0.022898"/>
+    <inertia ixx="0.000017128826"
+             iyy="0.000011930401"
+             izz="0.000008715513"
+             ixy="-0.000001953953"
+             iyz="0.00"
+             ixz="-0.00"/>
+  </inertial>
+  <visual>
+    <origin xyz="0.018 -0.719499 -0.0" rpy="0 0 0"/>
+    <geometry>
+      <mesh filename="package://amir_description/meshes/finger_left_1.stl" scale="0.001 0.001 0.001"/>
+    </geometry>
+    <material name="silver-amir"/>
+  </visual>
+  <collision>
+    <origin xyz="0.018 -0.719499 -0.0" rpy="0 0 0"/>
+    <geometry>
+      <mesh filename="package://amir_description/meshes/finger_left_1.stl" scale="0.001 0.001 0.001"/>
+    </geometry>
+  </collision>
+</link>
+<!-- end of inner link -->
+<!-- use this when using outer link -->
+<!-- <link name="finger_right_1">
+  <inertial>
+    <origin xyz="-0.01751055591310643 0.012411313372935995 0.0" rpy="0 0 0"/>
+    <mass value="0.08357364665097004"/>
+    <inertia ixx="6.7e-05" iyy="4.7e-05" izz="3.5e-05" ixy="8e-06" iyz="0.0" ixz="-0.0"/>
+  </inertial>
+  <visual>
+    <origin xyz="-0.038 -0.719499 -0.0" rpy="0 0 0"/>
+    <geometry>
+      <mesh filename="package://amir_description/meshes/finger_right_1.stl" scale="0.001 0.001 0.001"/>
+    </geometry>
+    <material name="silver-amir"/>
+  </visual>
+  <collision>
+    <origin xyz="-0.038 -0.719499 -0.0" rpy="0 0 0"/>
+    <geometry>
+      <mesh filename="package://amir_description/meshes/finger_right_1.stl" scale="0.001 0.001 0.001"/>
+    </geometry>
+  </collision>
+</link>
+<link name="finger_left_1">
+  <inertial>
+    <origin xyz="0.017510555913102525 0.012411313372938326 0.0" rpy="0 0 0"/>
+    <mass value="0.08357364665097004"/>
+    <inertia ixx="6.7e-05" iyy="4.7e-05" izz="3.5e-05" ixy="-8e-06" iyz="-0.0" ixz="-0.0"/>
+  </inertial>
+  <visual>
+    <origin xyz="0.038 -0.719499 -0.0" rpy="0 0 0"/>
+    <geometry>
+      <mesh filename="package://amir_description/meshes/finger_left_1.stl" scale="0.001 0.001 0.001"/>
+    </geometry>
+    <material name="silver-amir"/>
+  </visual>
+  <collision>
+    <origin xyz="0.038 -0.719499 -0.0" rpy="0 0 0"/>
+    <geometry>
+      <mesh filename="package://amir_description/meshes/finger_left_1.stl" scale="0.001 0.001 0.001"/>
+    </geometry>
+  </collision>
+</link> -->
+<!-- end of outer link -->
 <link name="inner_link_right_1">
   <inertial>
-    <origin xyz="-0.00362629710068591 0.012517792510871706 -0.017383026433693875" rpy="0 0 0"/>
-    <mass value="0.03672285115716527"/>
-    <inertia ixx="2.9e-05" iyy="2.2e-05" izz="1e-05" ixy="0.0" iyz="4e-06" ixz="-1e-06"/>
-  </inertial>
-  <visual>
-    <origin xyz="-0.017633 -0.677976 -0.026403" rpy="0 0 0"/>
+    <origin xyz="-0.003238561697949489 0.01183851365994859 0.0" rpy="0 0 0"/>
+    <mass value="0.009152"/>
+    <inertia ixx="0.000006905758"
+             iyy="0.000005170951"
+             izz="0.000002372537"
+             ixy="0.000000349609"
+             iyz="0.000000273496"
+             ixz="-0.000000039247"/>
+  </inertial>
+  <visual>
+    <origin xyz="-0.018 -0.679499 -0.0" rpy="0 0 0"/>
     <geometry>
       <mesh filename="package://amir_description/meshes/inner_link_right_1.stl" scale="0.001 0.001 0.001"/>
@@ -139,5 +360,5 @@
   </visual>
   <collision>
-    <origin xyz="-0.017633 -0.677976 -0.026403" rpy="0 0 0"/>
+    <origin xyz="-0.018 -0.679499 -0.0" rpy="0 0 0"/>
     <geometry>
       <mesh filename="package://amir_description/meshes/inner_link_right_1.stl" scale="0.001 0.001 0.001"/>
@@ -145,185 +366,119 @@
   </collision>
 </link>
-<link name="inner_link_left_1">
-  <inertial>
-    <origin xyz="0.0047898187388998766 0.014750783106671883 -0.02749955283980449" rpy="0 0 0"/>
-    <mass value="0.03083975679211874"/>
-    <inertia ixx="2.4e-05" iyy="1.8e-05" izz="8e-06" ixy="0.0" iyz="-0.0" ixz="-0.0"/>
-  </inertial>
-  <visual>
-    <origin xyz="0.018367 -0.677976 -0.027903" rpy="0 0 0"/>
-    <geometry>
-      <mesh filename="package://amir_description/meshes/inner_link_left_1.stl" scale="0.001 0.001 0.001"/>
-    </geometry>
-    <material name="silver-amir"/>
-  </visual>
-  <collision>
-    <origin xyz="0.018367 -0.677976 -0.027903" rpy="0 0 0"/>
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