Commit message: edited amir_description

File: amir_description/urdf/amir_f120a.xacro (robot description, xacro)
@@ -2,5 +2,5 @@
 <robot name="amir_f120a" xmlns:xacro="http://www.ros.org/wiki/xacro">
  <!-- Include F120A rover URDF -->
-<xacro:include filename="$(find f120a_description)/urdf/f120a.xacro"/>
+<xacro:include filename="$(find megarover_description)/urdf/f120a_base_model.xacro"/>
  <!-- Include AMIR URDF -->
 <xacro:include filename="$(find amir_description)/urdf/amir_for_rover.xacro"/>

File: amir_description/urdf/amir_mega3.xacro (robot description, xacro)
@@ -2,9 +2,9 @@
 <robot name="amir_mega3" xmlns:xacro="http://www.ros.org/wiki/xacro">
  <!-- Include mega3 rover URDF -->
-<xacro:include filename="$(find mega3_description)/urdf/mega3.xacro"/>
+<xacro:include filename="$(find megarover_description)/urdf/mega3_base_model.xacro"/>
  <!-- Include AMIR URDF -->
 <xacro:include filename="$(find amir_description)/urdf/amir_for_rover.xacro"/>
 <joint name="base_fixed" type="fixed">
-  <origin xyz="0.0 0.0 0.393" rpy="0 0 0"/>
+  <origin xyz="0.0 0.03 0.398" rpy="0 0 0"/>
   <parent link="base_link"/>
   <child link="link0_1"/>
